File: Hardware/KiCAD/BioZ_front_end_V2_1/BioZ_front_end_V2_1.kicad_pcb (KiCad board)
At the start: 4 copper layers, 262.5 x 120.1 mm, 362 parts, among them J1 DC IN, J10 CH1 IN-, J11 CH2 Output Con, J12 CH1 Output Con, J13 CH2 Input Con, J14 CH1 Input Con, J15 STIM_PWR, J16 EXT_Stim, J17 USB_C_Receptacle_USB2.0, J18 STM32 IO, J19 Vmes+, J2 JTAG, J20 Vmes-, J21 Stim-, J22 Stim+, J23 Load, J24 Load2, J25 Scope 1, J26 Scope 2, J27 AWG1, J28 Scope 1, J29 AD2 EXT Conn, J3 Power, J30 AWG2, J31 Scope 2, J32 AD2 Conn, J33 UART, J4 CH2_PWR, J5 CH1_PWR, J6 EXT_stim, J7 CH2 IN+, J8 CH2 IN-, J9 CH1 IN+, K1 EE2-5NUH-L, K10 EE2-5NUH-L, K11 EE2-5NUH-L, K12 EE2-5NUH-L, K13 EE2-5NUH-L, K14 EE2-5NUH-L, K15 EE2-5NUH-L, K16 EE2-5NUH-L, K17 EE2-5NUH-L, K18 EE2-5NUH-L, K19 EE2-5NUH-L, K2 EE2-5NUH-L, K20 EE2-5NUH-L, K21 EE2-5NUH-L, K22 EE2-5NUH-L, K23 EE2-5NUH-L, K3 EE2-5NUH-L, K4 EE2-5NUH-L, K5 EE2-5NUH-L, K6 EE2-5NUH-L, K7 EE2-5NUH-L, K8 EE2-5NUH-L, K9 EE2-5NUH-L, Q1 CPH3462, Q10 CPH3462, Q11 CPH3462, Q12 CPH3462, Q13 CPH3462, Q14 CPH3462, Q15 CPH3462, Q16 PMT200EPEX, Q17 PMT200EPEX, Q18 CPH3462, Q19 CPH3462, Q2 CPH3462, Q20 CPH3462, Q21 CPH3462, Q22 CPH3462, Q23 CPH3462, Q24 CPH3462, Q25 CPH3462, Q3 CPH3462, Q4 CPH3462, Q5 CPH3462, Q6 CPH3462, Q7 CPH3462, Q8 CPH3462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

Commit message: update files
Parts:
- removed Q16, Q17: PMT200EPEX, Package_TO_SOT_SMD:SOT-223-3_TabPin2
- added Q26: PMT200EPEX, Package_TO_SOT_SMD:SOT-223-3_TabPin2, F.Cu at (93.3, 36.6)
- added Q27: PMT200EPEX, Package_TO_SOT_SMD:SOT-223-3_TabPin2, F.Cu at (93.3, 48.1)
- C80: value x -> 0.5pF
- R109: renamed from 47k1; value R79 -> 47k
- R56: value 5k6 -> 1k
- moved R56 53.9 mm to (98.0, 68.7)
- moved C79 0.85 mm to (94.5, 69.1)
Connections:
- R56 pad 1: Vout+ -> I_load-_Cout
- R56 pad 2: Vout- -> I_load_Cout
Routing:
- net Net-(Q26-Pad1): track 20.0 -> 9.91 mm
- net Vin_USB: track 42.2 -> 50.8 mm, vias 1 -> 2
- net Net-(Q27-Pad1): track 14.1 -> 6.83 mm
- net Vin_DC: track 34.8 -> 41.4 mm
- net I_load-_Cout: track 51.2 -> 57.2 mm
- net I_load_Cout: track 53.3 -> 55.5 mm
- net Vout-: track 117.9 -> 115.9 mm
- net GND: track 1993.8 -> 1995.0 mm
- net Vout+: track 82.8 -> 81.8 mm
Other:
- board text removed: "+15V"
- board text removed: "-15V"
