File: Hardware/KiCAD/BioZ_front_end_V2_1/BioZ_front_end_V2_1.sch (KiCad schematic (older format))
At the start: 360 parts, among them J1 DC IN, J10 CH1 IN-, J11 CH2 Output Con, J12 CH1 Output Con, J13 CH2 Input Con, J14 CH1 Input Con, J15 STIM_PWR, J16 EXT_Stim, J17 USB_C_Receptacle_USB2.0, J18 STM32 IO, J19 Vmes+, J2 JTAG, J20 Vmes-, J21 Stim-, J22 Stim+, J23 Load, J24 Load2, J25 Scope 1, J26 Scope 2, J27 AWG1, J28 Scope 1, J29 AD2 EXT Conn, J3 Power, J30 AWG2, J31 Scope 2, J32 AD2 Conn, J33 UART, J4 CH2_PWR, J5 CH1_PWR, J6 EXT_stim, J7 CH2 IN+, J8 CH2 IN-, J9 CH1 IN+, K1 EE2-5NUH-L, K10 EE2-5NUH-L, K11 EE2-5NUH-L, K12 EE2-5NUH-L, K13 EE2-5NUH-L, K14 EE2-5NUH-L, K15 EE2-5NUH-L, K16 EE2-5NUH-L, K17 EE2-5NUH-L, K18 EE2-5NUH-L, K19 EE2-5NUH-L, K2 EE2-5NUH-L, K20 EE2-5NUH-L, K21 EE2-5NUH-L, K22 EE2-5NUH-L, K23 EE2-5NUH-L, K3 EE2-5NUH-L, K4 EE2-5NUH-L, K5 EE2-5NUH-L, K6 EE2-5NUH-L, K7 EE2-5NUH-L, K8 EE2-5NUH-L, K9 EE2-5NUH-L, Q1 CPH3462, Q10 CPH3462, Q11 CPH3462, Q12 CPH3462, Q13 CPH3462, Q14 CPH3462, Q15 CPH3462, Q16 PMT200EPEX, Q17 PMT200EPEX, Q18 CPH3462, Q19 CPH3462, Q2 CPH3462, Q20 CPH3462, Q21 CPH3462, Q22 CPH3462, Q23 CPH3462, Q24 CPH3462, Q25 CPH3462, Q3 CPH3462, Q4 CPH3462, Q5 CPH3462, Q6 CPH3462, Q7 CPH3462, Q8 CPH3462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

Commit message: update files
Parts:
- removed Q16, Q17: PMT200EPEX, Package_TO_SOT_SMD:SOT-223-3_TabPin2, symbol Device:Q_PMOS_DGS
- added Q26, Q27: PMT200EPEX, Package_TO_SOT_SMD:SOT-223-3_TabPin2, symbol Device:Q_PMOS_GDS
- C80: value x -> 0.5pF
- R56: value 5k6 -> 1k
Connections:
- wire segments 1153 -> 1154
Other:
- moved on the sheet: R57
Changed lines of the file:
@@
 	0    -1   -1   0
 $EndComp
-$Comp
-L Device:R R56
-U 1 1 70C55CE2
-P 10250 6950
-F 0 "R56" H 10320 6996 50  0000 L CNN
-F 1 "5k6" H 10320 6905 50  0000 L CNN
-F 2 "Resistor_SMD:R_0603_1608Metric" V 10180 6950 50  0001 C CNN
-F 3 "~" H 10250 6950 50  0001 C CNN
-	1    10250 6950
-	1    0    0    -1
-$EndComp
-Wire Wire Line
-	9550 6800 10250 6800
-Connection ~ 10250 6800
-Wire Wire Line
-	10250 6800 10650 6800
-Wire Wire Line
-	10250 7100 10650 7100
-Connection ~ 10250 7100
 Text GLabel 10650 6800 2    50   Input ~ 0
 Vout+
@@
 L power:GND #PWR0172
 U 1 1 74845BD2
-P 14650 3200
-F 0 "#PWR0172" H 14650 2950 50  0001 C CNN
-F 1 "GND" H 14655 3027 50  0000 C CNN
-F 2 "" H 14650 3200 50  0001 C CNN
-F 3 "" H 14650 3200 50  0001 C CNN
-	1    14650 3200
+P 14450 3200
+F 0 "#PWR0172" H 14450 2950 50  0001 C CNN
+F 1 "GND" H 14455 3027 50  0000 C CNN
+F 2 "" H 14450 3200 50  0001 C CNN
+F 3 "" H 14450 3200 50  0001 C CNN
+	1    14450 3200
 	1    0    0    -1
 $EndComp
@@
 L Device:R R57
 U 1 1 74845B7B
-P 14650 3000
-F 0 "R57" H 14720 3046 50  0000 L CNN
-F 1 "1M" H 14720 2955 50  0000 L CNN
-F 2 "Resistor_SMD:R_0603_1608Metric" V 14580 3000 50  0001 C CNN
-F 3 "~" H 14650 3000 50  0001 C CNN
-	1    14650 3000
+P 14450 3000
+F 0 "R57" H 14520 3046 50  0000 L CNN
+F 1 "1M" H 14520 2955 50  0000 L CNN
+F 2 "Resistor_SMD:R_0603_1608Metric" V 14380 3000 50  0001 C CNN
+F 3 "~" H 14450 3000 50  0001 C CNN
+	1    14450 3000
 	1    0    0    -1
 $EndComp
@@
 	14300 2850 14450 2850
 Connection ~ 14450 2850
-Wire Wire Line
-	14450 2850 14650 2850
 $Comp
 L power:+5V #PWR0212
@@
 $EndComp
 $Comp
-L Device:Q_PMOS_DGS Q17
-U 1 1 6335F035
-P 30850 7100
-F 0 "Q17" V 31099 7100 50  0000 C CNN
-F 1 "PMT200EPEX" V 31190 7100 50  0000 C CNN
-F 2 "Package_TO_SOT_SMD:SOT-223-3_TabPin2" H 31050 7200 50  0001 C CNN
-F 3 "~" H 30850 7100 50  0001 C CNN
-	1    30850 7100
-	0    -1   1    0
-$EndComp
-$Comp
-L Device:Q_PMOS_DGS Q16
-U 1 1 63450122
-P 30850 5750
-F 0 "Q16" V 31192 5750 50  0000 C CNN
-F 1 "PMT200EPEX" V 31101 5750 50  0000 C CNN
-F 2 "Package_TO_SOT_SMD:SOT-223-3_TabPin2" H 31050 5850 50  0001 C CNN
-F 3 "~" H 30850 5750 50  0001 C CNN
-	1    30850 5750
-	0    -1   -1   0
-$EndComp
-$Comp
 L Connector:USB_C_Receptacle_USB2.0 J17
 U 1 1 63451637
@@
 $EndComp
 Wire Wire Line
-	9550 7100 10250 7100
-Wire Wire Line
 	9250 7100 9150 7100
 Wire Wire Line
@@
 Wire Wire Line
 	14400 3500 14400 3900
-Wire Wire Line
-	14650 3150 14650 3200
-Wire Wire Line
-	14650 2850 15100 2850
-Connection ~ 14650 2850
 Connection ~ 15100 2850
 Wire Wire Line
 	15100 2850 15100 3100
 Wire Wire Line
-	14400 3500 15100 3500
+	14400 3500 14800 3500
 Connection ~ 14400 3500
 Wire Wire Line
@@
 P 16100 4200
 F 0 "C80" V 15848 4200 50  0000 C CNN
-F 1 "x" V 15939 4200 50  0000 C CNN
+F 1 "0.5pF" V 15939 4200 50  0000 C CNN
 F 2 "Capacitor_SMD:C_0603_1608Metric" H 16138 4050 50  0001 C CNN
 F 3 "~" H 16100 4200 50  0001 C CNN
@@
 	1    0    0    -1
 $EndComp
+Wire Wire Line
+	9550 6800 10650 6800
+Wire Wire Line
+	9550 7100 10650 7100
+$Comp
+L Device:R R56
+U 1 1 61EEF21F
+P 14800 3150
+F 0 "R56" V 15007 3150 50  0000 C CNN
+F 1 "1k" V 14916 3150 50  0000 C CNN
+F 2 "Resistor_SMD:R_0603_1608Metric" V 14730 3150 50  0001 C CNN
+F 3 "~" H 14800 3150 50  0001 C CNN
+	1    14800 3150
+	1    0    0    -1
+$EndComp
+Wire Wire Line
+	14450 3150 14450 3200
+Wire Wire Line
+	14450 2850 14800 2850
+Wire Wire Line
+	14800 2850 14800 3000
+Connection ~ 14800 2850
+Wire Wire Line
+	14800 2850 15100 2850
+Wire Wire Line
+	14800 3300 14800 3500
+Connection ~ 14800 3500
+Wire Wire Line
+	14800 3500 15100 3500
+$Comp
+L Device:Q_PMOS_GDS Q26
+U 1 1 6259E97F
+P 30850 5750
+F 0 "Q26" V 31192 5750 50  0000 C CNN
+F 1 "PMT200EPEX" V 31101 5750 50  0000 C CNN
+F 2 "Package_TO_SOT_SMD:SOT-223-3_TabPin2" H 31050 5850 50  0001 C CNN
+F 3 "~" H 30850 5750 50  0001 C CNN
+	1    30850 5750
+	0    -1   -1   0
+$EndComp
+$Comp
+L Device:Q_PMOS_GDS Q27
+U 1 1 625A5686
+P 30850 7100
+F 0 "Q27" V 31099 7100 50  0000 C CNN
+F 1 "PMT200EPEX" V 31190 7100 50  0000 C CNN
+F 2 "Package_TO_SOT_SMD:SOT-223-3_TabPin2" H 31050 7200 50  0001 C CNN
+F 3 "~" H 30850 7100 50  0001 C CNN
+	1    30850 7100
+	0    -1   1    0
+$EndComp
 $EndSCHEMATC
